File: PCB-MAIN/Main/Main.kicad_sch (KiCad schematic)
At the start: 45 parts, among them J1 Conn_01x02, J10 UART-OUT, J11 Conn_01x02, J12 Conn_01x02, J13 Conn_01x01_Shielded, J14 Conn_01x04, J15 SERVO-OUT-1, J16 216701-0609, J17 SERVO-OUT-2, J18 BUS-DEBUG, J19 JTAG, J2 USB-C, J20 Conn_01x02, J3 Conn_01x02, J4 Conn_01x02, J5 Conn_01x02, J6 216700-0609, J7 Conn_01x02, J8 Conn_01x02, J9 Conn_01x02, Q1 Q_NMOS_GSD, Q10 Q_NMOS_GSD, Q2 Q_NMOS_GSD, Q3 Q_NMOS_GSD, Q4 Q_NMOS_GSD, Q5 Q_NMOS_GSD, Q6 Q_NMOS_GSD, Q7 Q_NMOS_GSD, Q8 Q_NMOS_GSD, Q9 Q_NMOS_GSD, U1 F28P550SG8PNAR, U10 LTE3401LX, U11 MIC2876, U12 ICP-10111, U12 IS25LP040E-JYLE-TR, U13 NX3DV221TKX, U14 NCV7344AD10R2G, U15 NCV7344AD10R2G, U2 LSM6DS3, U3 KX122-1042, U4 STM32WL33KBV6, U6 SC0914_13_, U7 LTE3401LX, U9 AP61402, Y1 Crystal_GND24_Small

Commit message: helper scripts and finishing the digital circuitry, working now on power domain
Parts:
- removed J18: BUS-DEBUG, Connector_PinSocket_2.54mm:PinSocket_2x05_P2.54mm_Vertical, symbol Connector_Generic:Conn_02x05_Top_Bottom
- added D1: BAS16TS_R1_00001, Diode_SMD:D_SOD-523, symbol Diode:BAS516
- added J18: UART-OUT, Connector_PinHeader_2.54mm:PinHeader_1x04_P2.54mm_Vertical, symbol Connector_Generic:Conn_01x04
- added J21: DEBUG, Connector_PinHeader_2.54mm:PinHeader_2x07_P2.54mm_Vertical, symbol Connector_Generic:Conn_02x07_Odd_Even
- added TP1: TestPoint_2Pole, Connector_PinSocket_1.00mm:PinSocket_1x02_P1.00mm_Vertical_SMD_Pin1Left, symbol Connector:TestPoint_2Pole
- added TP2, TP3: TestPoint, TestPoint:TestPoint_Pad_D1.0mm, symbol Connector:TestPoint
- added U5: CD74HC4067SM, Package_SO:SSOP-24_5.3x8.2mm_P0.65mm, symbol 74xx:CD74HC4067SM
- J14: value Conn_01x04 -> Conn_DEBUG_1
Connections:
- net +3V3: now also J10.3 (Pin_3), J19.13 (Pin_13), U12.8 (VCC), U12.8 (VDD), U14.3 (VCC), U15.3 (VCC), U2.5 (VDDIO), U2.8 (VDD), U3.3 (IO_VDD), U3.7 (VDD), J18.1 (Pin_1)
- net GND: now also J1.2 (Pin_2), J10.4 (Pin_4), J19.14 (Pin_14), Q10.2 (S), Q3.2 (S), Q4.2 (S), Q5.2 (S), Q6.2 (S), Q7.2 (S), Q8.2 (S), Q9.2 (S), U1.16 (A11), U1.17 (A5), U1.22 (A12), U1.23 (A7), U1.24 (A8), U11.2 (PGND), U11.4 (AGND), U12.1 (GND_1), U12.2 (RESV_1), U12.5 (RESV_2), U12.6 (RESV_3), U12.7 (GND_2), U13.11 (EP), U13.5 (GND), U14.2 (GND), U15.2 (GND), U2.6 (GND), U2.7 (GND), U3.9 (GND), U4.33 (EP), U6.19 (TESTEN), U9.4 (GND), J18.4 (Pin_4), U5.12 (GND)
- net +BATT: now reaches U9.6 (VIN)
- net +BATT: now also J1.1 (Pin_1), U11.3 (IN)
- net at U1.14 (A15): now also J16.4
- net at U1.28 (GPIO236): now also J21.3 (Pin_3)
- net at U1.29 (GPIO230): now also J21.5 (Pin_5)
- net at U1.31 (GPIO62): now also J21.7 (Pin_7)
- net at U1.32 (GPIO63): now also J21.9 (Pin_9)
- net at U1.33 (GPIO20): now also J21.11 (Pin_11)
- net at U1.34 (GPIO21): now also J21.13 (Pin_13)
- net at U1.35 (GPIO13): now also J16.36
- net at U1.37 (GPIO11): now also J16.28; no longer J16.36
- net at U1.41 (GPIO24): now also J21.2 (Pin_2); no longer J16.28
- net at U1.54 (GPIO43): now also J21.1 (Pin_1)
- net at U1.57 (GPIO42): now also J21.4 (Pin_4)
- net at U1.64 (GPIO40): now also TP3.1
- net at U1.67 (GPIO22): now also TP2.1
- net at U1.68 (GPIO7): now also J21.14 (Pin_14)
- net at U1.69 (GPIO44): now also J21.12 (Pin_12)
- net at U1.73 (GPIO45): now also J21.10 (Pin_10)
- net at U1.74 (GPIO5): now also J21.8 (Pin_8)
- net at U1.75 (GPIO9): now also J21.6 (Pin_6)
- net at U2.4 (INT1): now also U5.18 (I13)
- net at U2.9 (INT2): now also U5.19 (I12)
- net at J10.1 (Pin_1): now also J6.6
- net at J10.2 (Pin_2): now also J6.5
- net at U4.1 (PA2), U6.31 (GPIO20): now also J14.3 (Pin_3), D1.2 (A); no longer Q10.1 (G)
- net at U3.4 (TRIG), U4.2 (PA3): now also J14.2 (Pin_2)
- net at U4.24 (NRST): now also J14.4 (Pin_4)
- net at U4.4 (PA0): now also J14.1 (Pin_1)
- net at Q7.1 (G): now also U5.6 (I3)
- net at U3.5 (INT1): now also U5.17 (I14)
- net at U3.6 (INT2): now also U5.16 (I15)
- net at Q8.1 (G): now also U5.7 (I2)
- net at Q6.1 (G): now also U5.5 (I4)
- net at U6.10 (IOVDD_2): now also U5.15 (~{E})
- net at U6.24 (SWCLK): now also J19.12 (Pin_12)
- net at U6.25 (SWDIO): now also J19.11 (Pin_11)
- net at U6.26 (RUN): now also J19.10 (Pin_10)
- net at J19.1 (Pin_1): now also J6.46
- net at J19.2 (Pin_2): now also J6.43
- net at J19.3 (Pin_3): now also J6.48
- net at J19.4 (Pin_4): now also J6.47
- net at J19.5 (Pin_5): now also J6.50
- net at J19.6 (Pin_6): now also J6.49
- net at J19.7 (Pin_7): now also J6.52
- net at J19.8 (Pin_8): now also J6.51
- net at J19.9 (Pin_9): now also J6.42
- net at Q9.1 (G): now also U5.8 (I1)
- net at Q4.1 (G): now also U5.3 (I6)
- net at U15.1 (TXD): now also J6.36
- net at U15.4 (RXD): now also J6.35
- net at U15.6 (CANL): now also U14.6 (CANL), J18.3 (Pin_3)
- net at U15.7 (CANH): now also U14.7 (CANH), J18.2 (Pin_2)
- net at U15.8 (STB): now also U5.20 (I11)
- net at Q3.1 (G): now also U5.2 (I7)
- net at J6.12: now also U5.1 (COM)
- net at J6.13: now also U5.10 (S0)
- net at J6.14: now also U5.11 (S1)
- net at J6.15: now also U5.14 (S2)
- net at J6.16: now also U5.13 (S3)
- net at Q5.1 (G): now also U5.4 (I5)
- new net: D1.1 (K), Q10.1 (G), U5.9 (I0)
Other:
- note added: "ADC channels"
- note added: "ADCE_SEL"
- note added: "CAN Bus"
- note added: "Clocks"
- note added: "Debug"
- note added: "I2C Bus"
- note added: "OUTPUTXBAR"
- note added: "SPI Bus"
- note added: "UART"
- note added: "USB"
- moved on the sheet: J1, J14, J16, J19, J2, U1, U11, U15, U9
